Commit message: Implemented launch file for gazebo; gazebo fully running; debugging controller manager startup issue

File: src/furi_description/urdf/dobot_magician_lite.urdf.xacro (robot description, xacro)
@@ -1,4 +1,10 @@
 <?xml version="1.0"?>
+<!-- Stage 4 Gazebo simulation control.
+      Position commands are provided by ros2_control through Gazebo.
+      The existing FURI software pipeline still owns:
+      /furi/command/raw -> /furi/command/applied -> simulated robot.
+-->
 <robot xmlns:xacro="http://www.ros.org/wiki/xacro" name="dobot_magician_lite">
+  <xacro:arg name="controllers_file" default=""/>
   <!--
     Dobot Magician Lite software-only kinematic model.
@@ -17,5 +23,4 @@
     - J3: -10 to +85 deg
     - J4: -145 to +145 deg
-    This is a clean educational model for software validation.
     Refine link mesh geometry later after measuring the physical arm.
   -->
@@ -226,3 +231,49 @@
     </inertial>
   </link>
+  <gazebo>
+    <plugin name="gazebo_ros2_control" filename="libgazebo_ros2_control.so">
+      <parameters>$(arg controllers_file)</parameters>
+    </plugin>
+  </gazebo>
+  <ros2_control name="GazeboSystem" type="system">
+    <hardware>
+      <plugin>gazebo_ros2_control/GazeboSystem</plugin>
+    </hardware>
+    <joint name="joint_1">
+      <command_interface name="position">
+        <param name="min">${j1_lower}</param>
+        <param name="max">${j1_upper}</param>
+      </command_interface>
+      <state_interface name="position"/>
+      <state_interface name="velocity"/>
+      <state_interface name="effort"/>
+    </joint>
+    <joint name="joint_2">
+      <command_interface name="position">
+        <param name="min">${j2_lower}</param>
+        <param name="max">${j2_upper}</param>
+      </command_interface>
+      <state_interface name="position"/>
+      <state_interface name="velocity"/>
+      <state_interface name="effort"/>
+    </joint>
+    <joint name="joint_3">
+      <command_interface name="position">
+        <param name="min">${j3_lower}</param>
+        <param name="max">${j3_upper}</param>
+      </command_interface>
+      <state_interface name="position"/>
+      <state_interface name="velocity"/>
+      <state_interface name="effort"/>
+    </joint>
+    <joint name="joint_4">
+      <command_interface name="position">
+        <param name="min">${j4_lower}</param>
+        <param name="max">${j4_upper}</param>
+      </command_interface>
+      <state_interface name="position"/>
+      <state_interface name="velocity"/>
+      <state_interface name="effort"/>
+    </joint>
+  </ros2_control>
 </robot>

Commit message: Implemented Gazebo launch pipeline and tested simulation joint constraints

File: src/furi_description/urdf/dobot_magician_lite.urdf.xacro (robot description, xacro)
@@ -1,5 +1,5 @@
 <?xml version="1.0"?>
 <!-- Stage 4 Gazebo simulation control.
-      Position commands are provided by ros2_control through Gazebo.
+      Position commands (rad) are adapted from FURI velocities by sim_robot_bridge.
       The existing FURI software pipeline still owns:
       /furi/command/raw -> /furi/command/applied -> simulated robot.
@@ -7,11 +7,12 @@
 <robot xmlns:xacro="http://www.ros.org/wiki/xacro" name="dobot_magician_lite">
   <xacro:arg name="controllers_file" default=""/>
+  <xacro:arg name="enable_gazebo" default="false"/>
   <!--
     Dobot Magician Lite software-only kinematic model.
     Purpose:
     - Stage 3: URDF/Xacro, TF tree, RViz visualization, and kinematic sanity checks.
-    - No Gazebo plugins.
+    - Optional Gazebo Classic control enabled only by the simulation launch.
+    - Approximate masses, inertias and effort limits; no calibrated dynamics.
     - No hardware drivers.
-    - No ros2_control yet.
     Main public specs used:
     - 4 DOF
@@ -121,4 +122,6 @@
     </inertial>
   </link>
+  <!-- Positive simulation pitch lifts the arm above the tabletop. Hardware
+       angle conventions and the real parallelogram linkage are not modeled. -->
   <!-- J2 shoulder pitch -->
   <joint name="joint_2" type="revolute">
@@ -126,5 +129,5 @@
     <child link="upper_arm_link"/>
     <origin xyz="0 0 ${shoulder_height}" rpy="0 0 0"/>
-    <axis xyz="0 1 0"/>
+    <axis xyz="0 -1 0"/>
     <limit lower="${j2_lower}" upper="${j2_upper}" effort="${j_effort}" velocity="${j123_velocity}"/>
   </joint>
@@ -154,5 +157,5 @@
     <child link="forearm_link"/>
     <origin xyz="${upper_arm_length} 0 0" rpy="0 0 0"/>
-    <axis xyz="0 1 0"/>
+    <axis xyz="0 -1 0"/>
     <limit lower="${j3_lower}" upper="${j3_upper}" effort="${j_effort}" velocity="${j123_velocity}"/>
   </joint>
@@ -231,6 +234,18 @@
     </inertial>
   </link>
+  <xacro:if value="$(arg enable_gazebo)">
+  <!-- Mount the tabletop robot without making the articulated links static. -->
+  <link name="world"/>
+  <joint name="world_mount" type="fixed">
+    <parent link="world"/>
+    <child link="base_footprint"/>
+  </joint>
   <gazebo>
     <plugin name="gazebo_ros2_control" filename="libgazebo_ros2_control.so">
+      <robot_param>robot_description</robot_param>
+      <robot_param_node>robot_state_publisher</robot_param_node>
+      <controller_manager_name>controller_manager</controller_manager_name>
+      <hold_joints>true</hold_joints>
+      <ros><namespace>/</namespace></ros>
       <parameters>$(arg controllers_file)</parameters>
     </plugin>
@@ -277,3 +292,4 @@
     </joint>
   </ros2_control>
+  </xacro:if>
 </robot>
